File: Power_schematics.kicad_sch (KiCad schematic)
At the start: 27 parts, among them Q3 FS8205A, Q4 AO3401A, U5 DW01A

Commit message: version 1.1
Parts:
- added D12: Power LED, LED_SMD:LED_0603_1608Metric_Pad1.05x0.95mm_HandSolder, symbol Device:LED_Small
- added R1: 330, Resistor_SMD:R_0603_1608Metric_Pad0.98x0.95mm_HandSolder, symbol Device:R_Small
- added SW6: SW_SPDT, TP4056:SW_spdt _slide, symbol Switch:SW_SPDT
- Q3: footprint Package_SO:TSSOP-8_3x3mm_P0.65mm -> Package_SO:TSSOP-8_4.4x3mm_P0.65mm
- U?: footprint Package_TO_SOT_SMD:TO-252-3_TabPin2 -> Package_TO_SOT_SMD:SOT-223
Connections:
- net +3.3V: now also U?.4, R1.1
- net GND: now also D12.1 (K)
- net VOUT+: now also SW6.2 (B); no longer D11.1 (K), Q4.2 (S)
- net at Q3.1: no longer Q3.8
- new net: D11.1 (K), Q4.2 (S), SW6.1 (A)
- new net: D12.2 (A), R1.2
- no-connect marks 2 -> 3
