File: Conn_schematics.kicad_sch.kicad_sch (KiCad schematic)
At the start: 37 parts, among them J1 SPI, J10 GNDS, J2 CSP-USC16-TR, J3 I2c, J4 UART2, J5 Motor A, J6 Motor B, J7 DAC & ADC, J8 JTAG, J9 Conn_01x01

Commit message: version 1.1
Parts:
- removed BT1: BK-18650-PC2, BK-18650-PC2:BAT_BK-18650-PC2, symbol BK-18650-PC2:BK-18650-PC2
- removed J10: GNDS, Connector_PinHeader_2.54mm:PinHeader_1x02_P2.54mm_Vertical, symbol Connector_Generic:Conn_01x02
- removed J2: CSP-USC16-TR, CSP-USC16-TR:VALCON_CSP-USC16-TR, symbol CSP-USC16-TR:CSP-USC16-TR
- removed R? (x2): 5k1, Resistor_SMD:R_0603_1608Metric_Pad0.98x0.95mm_HandSolder, symbol Device:R_Small
- added J13: Battery, TP4056:connector_2pin_5.08, symbol Connector_Generic:Conn_01x02
- added U8: ~, TP4056:TypeC_254, symbol TP4056:TypeC254
Connections:
- net +3.3V: now also J1.0 (Pin_1), J3.0 (Pin_1), J4.0 (Pin_1), J7.0 (Pin_1)
- net +5V: now also U8.4 (Vcc)
- net BATCONN+: now also J13.1 (Pin_1)
- net BATCONN-: now also J13.2 (Pin_2)
- net D+: now also U8.2 (D+)
- net D-: now also U8.3 (D-)
- net GND: now also U8.1 (GND)
- no-connect marks 2 -> 0
Other:
- note removed: "GND points"

Commit message: edited
Parts:
- removed D?: GREEN, LED_SMD:LED_0603_1608Metric_Pad1.05x0.95mm_HandSolder, symbol Device:LED_Small
- removed R?: 330, Resistor_SMD:R_0603_1608Metric_Pad0.98x0.95mm_HandSolder, symbol Device:R_Small
Changed lines of the file:
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@@
-    (stroke (width 0) (type default))
-  )
-  (wire (pts (xy 203.2 27.94) (xy 203.2 31.75))
     (stroke (width 0) (type default))
   )
@@
     (stroke (width 0) (type default))
   )
-  (wire (pts (xy 200.66 50.8) (xy 203.2 50.8))
-    (stroke (width 0) (type default))
-  )
   (wire (pts (xy 45.72 132.08) (xy 57.15 132.08))
     (stroke (width 0) (type default))
@@
     (stroke (width 0) (type default))
   )
-  (wire (pts (xy 203.2 50.8) (xy 203.2 44.45))
-    (stroke (width 0) (type default))
-  )
   (wire (pts (xy 231.14 100.33) (xy 231.14 102.87))
     (stroke (width 0) (type default))
@@
   )
   (wire (pts (xy 109.22 46.99) (xy 109.22 50.8))
-    (stroke (width 0) (type default))
-  )
-  (wire (pts (xy 203.2 36.83) (xy 203.2 39.37))
     (stroke (width 0) (type default))
   )
@@
     (effects (font (size 2 2)) (justify left bottom))
   )
-  (text "LED outputs\n" (at 191.77 19.05 0)
+  (text "LED outputs\n" (at 215.9 19.05 0)
     (effects (font (size 2 2)) (justify left bottom))
   )
@@
     )
   )
-  (global_label "GIO_23" (shape input) (at 200.66 50.8 180) (fields_autoplaced)
-    (effects (font (size 1.27 1.27)) (justify right))
-    (property "Intersheetrefs" "${INTERSHEET_REFS}" (at 191.0829 50.8 0)
-      (effects (font (size 1.27 1.27)) (justify right) hide)
-    )
-  )
   (global_label "GIO_17" (shape input) (at 85.09 184.15 270) (fields_autoplaced)
     (effects (font (size 1.27 1.27)) (justify right))
@@
     )
   )
-  (symbol (lib_id "Device:R_Small") (at 203.2 34.29 0) (unit 1)
-    (in_bom yes) (on_board yes) (dnp no) (fields_autoplaced)
-    (property "Reference" "R?" (at 205.74 33.02 0)
-      (effects (font (size 1.27 1.27)) (justify left))
-    )
-    (property "Value" "330" (at 205.74 35.56 0)
-      (effects (font (size 1.27 1.27)) (justify left))
-    )
-    (property "Footprint" "Resistor_SMD:R_0603_1608Metric_Pad0.98x0.95mm_HandSolder" (at 203.2 34.29 0)
-      (effects (font (size 1.27 1.27)) hide)
-    )
-    (property "Datasheet" "~" (at 203.2 34.29 0)
-      (effects (font (size 1.27 1.27)) hide)
-    )
-    (pin "1")
-    (pin "2")
-    (instances
-      (project "ESPCARproject"
-        (path "/2f4c7fe4-d81d-42af-a8ed-35cbf01f7760/33af9e60-1f78-4455-a2ff-f16cbea40dbc"
-          (reference "R?") (unit 1)
-        )
-        (path "/2f4c7fe4-d81d-42af-a8ed-35cbf01f7760/4d4dbb73-9fbe-4eda-9dd2-50ab8968a5d5"
-          (reference "R3") (unit 1)
-        )
-      )
-    )
-  )
   (symbol (lib_id "Switch:SW_Push") (at 214.63 95.25 90) (unit 1)
     (in_bom yes) (on_board yes) (dnp no)
@@
     )
   )
-  (symbol (lib_id "Device:LED_Small") (at 203.2 41.91 90) (unit 1)
-    (in_bom yes) (on_board yes) (dnp no)
-    (property "Reference" "D?" (at 201.93 39.37 0)
-      (effects (font (size 1.27 1.27)))
-    )
-    (property "Value" "GREEN" (at 200.66 45.72 0)
-      (effects (font (size 1.27 1.27)))
-    )
-    (property "Footprint" "LED_SMD:LED_0603_1608Metric_Pad1.05x0.95mm_HandSolder" (at 203.2 41.91 90)
-      (effects (font (size 1.27 1.27)) hide)
-    )
-    (property "Datasheet" "~" (at 203.2 41.91 90)
-      (effects (font (size 1.27 1.27)) hide)
-    )
-    (pin "1")
-    (pin "2")
-    (instances
-      (project "ESPCARproject"
-        (path "/2f4c7fe4-d81d-42af-a8ed-35cbf01f7760/33af9e60-1f78-4455-a2ff-f16cbea40dbc"
-          (reference "D?") (unit 1)
-        )
-        (path "/2f4c7fe4-d81d-42af-a8ed-35cbf01f7760/4d4dbb73-9fbe-4eda-9dd2-50ab8968a5d5"
-          (reference "D4") (unit 1)
-        )
-      )
-    )
-  )
   (symbol (lib_id "Diode:ESD9B3.3ST5G") (at 109.22 43.18 90) (unit 1)
     (in_bom yes) (on_board yes) (dnp no)
@@
         )
       )
-    )
-  )
-  (symbol (lib_id "power:+3.3V") (at 203.2 27.94 0) (unit 1)
-    (in_bom yes) (on_board yes) (dnp no)
-    (property "Reference" "#PWR?" (at 203.2 31.75 0)
-      (effects (font (size 1.27 1.27)) hide)
-    )
-    (property "Value" "+3.3V" (at 203.2 22.86 0)
-      (effects (font (size 1.27 1.27)))
-    )
-    (property "Footprint" "" (at 203.2 27.94 0)
-      (effects (font (size 1.27 1.27)) hide)
-    )
-    (property "Datasheet" "" (at 203.2 27.94 0)
-      (effects (font (size 1.27 1.27)) hide)
-    )
-    (pin "1")
-    (instances
-      (project "ESPCARproject"
-        (path "/2f4c7fe4-d81d-42af-a8ed-35cbf01f7760/33af9e60-1f78-4455-a2ff-f16cbea40dbc"
-          (reference "#PWR?") (unit 1)
-        )
-        (path "/2f4c7fe4-d81d-42af-a8ed-35cbf01f7760/4d4dbb73-9fbe-4eda-9dd2-50ab8968a5d5"
-          (reference "#PWR017") (unit 1)
-        )
-      )
