File: ESPCARproject.kicad_pcb (KiCad board)
At the start: 2 copper layers, 78 x 92 mm, 102 parts, among them J1 SPI, J10 GNDS, J2 CSP-USC16-TR, J3 I2c, J4 UART2, J5 Motor A, J6 Motor B, J7 DAC & ADC, J8 JTAG, J9 Conn_01x01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

Commit message: version 1.1
Parts:
- removed BT1: BK-18650-PC2, BK-18650-PC2:BAT_BK-18650-PC2
- removed J10: GNDS, Connector_PinHeader_2.54mm:PinHeader_1x02_P2.54mm_Vertical
- removed J2: CSP-USC16-TR, CSP-USC16-TR:VALCON_CSP-USC16-TR
- removed R14: 1k, Resistor_SMD:R_0603_1608Metric_Pad0.98x0.95mm_HandSolder
- removed R15: 10k, Resistor_SMD:R_0603_1608Metric_Pad0.98x0.95mm_HandSolder
- removed R2: 5k1, Resistor_SMD:R_0603_1608Metric_Pad0.98x0.95mm_HandSolder
- removed R8: 22k1, Resistor_SMD:R_0603_1608Metric_Pad0.98x0.95mm_HandSolder
- removed R9: 47k5, Resistor_SMD:R_0603_1608Metric_Pad0.98x0.95mm_HandSolder
- removed U1: CP2102N-Axx-xQFN28, Package_DFN_QFN:QFN-28-1EP_5x5mm_P0.5mm_EP3.35x3.35mm
- added D12: Power LED, LED_SMD:LED_0603_1608Metric_Pad1.05x0.95mm_HandSolder, F.Cu at (169.9, 119.5)
- added J13: Battery, TP4056:connector_2pin_5.08, F.Cu at (149.3, 129.2)
- added SW6: SW_SPDT, TP4056:SW_spdt _slide, F.Cu at (174.3, 138.6)
- added U7: CH340C, Package_SO:SOIC-16_3.9x9.9mm_P1.27mm, F.Cu at (116.9, 91.1)
- added U8: ~, TP4056:TypeC_254, F.Cu at (111.7, 140.3)
- Q3: footprint Package_SO:TSSOP-8_3x3mm_P0.65mm -> Package_SO:TSSOP-8_4.4x3mm_P0.65mm
- R1: value 5k1 -> 330
- U6: footprint Package_TO_SOT_SMD:TO-252-3_TabPin2 -> Package_TO_SOT_SMD:SOT-223
- moved R1 57.4 mm to (165.9, 119.5), turned to 0 degrees
- moved J6 52.6 mm to (163.4, 129.2), turned to 180 degrees
- moved D3 42.3 mm to (111.0, 122.7)
- moved C1 41.1 mm to (113.1, 122.3)
- moved D1 39.6 mm to (119.9, 123.1), turned to 180 degrees
- moved D2 38.4 mm to (116.0, 123.1), turned to 0 degrees
- moved J5 35.1 mm to (134.7, 129.2), turned to 180 degrees
- moved J7 18.1 mm to (183.6, 104.0)
- moved R23 17.6 mm to (165.1, 76.8), turned to 180 degrees
- moved R24 15.8 mm to (165.1, 78.9), turned to 180 degrees
- moved C25 15.6 mm to (174.7, 116.6), turned to 0 degrees
- moved R36 15.1 mm to (150.3, 107.6), turned to -90 degrees
- moved J4 13.9 mm to (183.6, 90.1)
- moved C7 9.37 mm to (116.5, 85.2)
- moved J1 9.20 mm to (183.6, 70.8)
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Connections:
- D11 pad 1: VOUT+ -> Net-(D11-K)
- Q3 pad 8: unconnected-(Q3-Pad1) -> unconnected-(Q3-Pad8)
- Q4 pad 2: VOUT+ -> Net-(D11-K)
- R1 pad 1: Net-(J2-CC1) -> +3.3V
- R1 pad 2: GND -> Net-(D12-A)
Routing:
- net +5V: track 159.9 -> 214.6 mm, vias 8 -> 2
- net BATCONN-: track 92.2 -> 42.5 mm, vias 1 -> 0
- net Net-(D11-K): track 0.00 -> 48.5 mm
- net +3.3V: track 125.7 -> 89.7 mm, vias 34 -> 28
- net D+: track 20.8 -> 47.8 mm, vias 2 -> 0
- net D-: track 21.4 -> 47.7 mm
- net VOUT+: track 89.0 -> 108.5 mm
- net /MCU/RXD: track 5.76 -> 25.1 mm
- net GIO_35: track 74.2 -> 92.1 mm
- net GIO_34: track 72.5 -> 90.4 mm
- net /MCU/TXD: track 8.36 -> 25.1 mm
- net AO1: track 43.5 -> 58.7 mm, vias 0 -> 1
- net GIO_17: track 42.6 -> 57.4 mm
- net GIO_25: track 73.9 -> 88.3 mm
- net RTS: track 68.9 -> 82.1 mm, vias 2 -> 3
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Other:
- board text added: "+"
- board text added: "-"
- board text added: "ADC/DAC"
- board text added: "Battery"
- board text added: "I2C"
- board text added: "JTAG"
- board text added: "MotorA"
- board text added: "MotorB"
- board text added: "NAND сургалтын төв машин загвар v1.1 2023"
- board text added: "Power SW"
- board text added: "SPI"
- board text added: "UART2"
- board text removed: "NAND сургалтын төв машин загвар v1.0"

Commit message: edited
Parts:
- removed D4: GREEN, LED_SMD:LED_0603_1608Metric_Pad1.05x0.95mm_HandSolder
- removed R17, R18, R19, R23: 10k, Resistor_SMD:R_0603_1608Metric_Pad0.98x0.95mm_HandSolder
- removed R3: 330, Resistor_SMD:R_0603_1608Metric_Pad0.98x0.95mm_HandSolder
- moved R4 2.43 mm to (125.9, 69.6)
- moved D5 2.43 mm to (131.2, 69.6)
Routing:
- net GIO_23: track 112.5 -> 105.6 mm
- net Net-(D4-A): track 3.54 -> 0.00 mm
- net +3.3V: track 89.7 -> 88.2 mm, vias 28 -> 27
- net GIO_5: track 69.9 -> 70.9 mm
