File: MCU_schematics.kicad_sch (KiCad schematic)
At the start: 39 parts, among them Q1 SS8050, Q2 SS8050, U7 CH340C

Commit message: version 1.1
Parts:
- removed R?: 47k5, Resistor_SMD:R_0603_1608Metric_Pad0.98x0.95mm_HandSolder, symbol Device:R_Small
- removed R?: 1k, Resistor_SMD:R_0603_1608Metric_Pad0.98x0.95mm_HandSolder, symbol Device:R_Small
- removed R?: 10k, Resistor_SMD:R_0603_1608Metric_Pad0.98x0.95mm_HandSolder, symbol Device:R_Small
- removed R?: 22k1, Resistor_SMD:R_0603_1608Metric_Pad0.98x0.95mm_HandSolder, symbol Device:R_Small
- removed U?: CP2102N-Axx-xQFN28, Package_DFN_QFN:QFN-28-1EP_5x5mm_P0.5mm_EP3.35x3.35mm, symbol Interface_USB:CP2102N-Axx-xQFN28
Connections:
- net +3.3V: now also U7.16 (VCC), U7.4 (V3)
- net D+: now also U7.5 (UD+)
- net D-: now also U7.6 (UD-)
- net DTR: now also U7.13 (~{DTR})
- net GND: now also U7.1 (GND)
- net RTS: now also U7.14 (~{RTS})
- net RXD: now also U7.3 (RXD)
- net TXD: now also U7.2 (TXD)
- no-connect marks 28 -> 17
Other:
- moved on the sheet: C?, U7

Commit message: edited
Parts:
- removed R? (x4): 10k, Resistor_SMD:R_0603_1608Metric_Pad0.98x0.95mm_HandSolder, symbol Device:R_Small
Changed lines of the file:
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@@
   (junction (at 38.1 31.75) (diameter 0) (color 0 0 0 0)
   )
-  (junction (at 102.87 165.1) (diameter 0) (color 0 0 0 0)
-  )
   (junction (at 266.7 48.26) (diameter 0) (color 0 0 0 0)
   )
@@
   (junction (at 266.7 33.02) (diameter 0) (color 0 0 0 0)
   )
-  (junction (at 99.06 181.61) (diameter 0) (color 0 0 0 0)
-  )
   (junction (at 157.48 129.54) (diameter 0) (color 0 0 0 0)
   )
@@
   (junction (at 68.58 31.75) (diameter 0) (color 0 0 0 0)
   )
-  (junction (at 106.68 162.56) (diameter 0) (color 0 0 0 0)
-  )
   (junction (at 223.52 144.78) (diameter 0) (color 0 0 0 0)
   )
   (junction (at 106.68 181.61) (diameter 0) (color 0 0 0 0)
   )
-  (junction (at 99.06 167.64) (diameter 0) (color 0 0 0 0)
-  )
   (junction (at 95.25 147.32) (diameter 0) (color 0 0 0 0)
   )
@@
   (junction (at 38.1 39.37) (diameter 0) (color 0 0 0 0)
   )
-  (junction (at 215.9 144.78) (diameter 0) (color 0 0 0 0)
-  )
   (junction (at 243.84 33.02) (diameter 0) (color 0 0 0 0)
   )
@@
   )
   (junction (at 129.54 130.81) (diameter 0) (color 0 0 0 0)
-  )
-  (junction (at 102.87 181.61) (diameter 0) (color 0 0 0 0)
   )
   (junction (at 114.3 154.94) (diameter 0) (color 0 0 0 0)
@@
     (stroke (width 0) (type default))
   )
-  (wire (pts (xy 102.87 177.8) (xy 102.87 181.61))
-    (stroke (width 0) (type default))
-  )
-  (wire (pts (xy 102.87 165.1) (xy 121.92 165.1))
+  (wire (pts (xy 86.36 165.1) (xy 121.92 165.1))
     (stroke (width 0) (type default))
   )
@@
     (stroke (width 0) (type default))
   )
-  (wire (pts (xy 106.68 162.56) (xy 121.92 162.56))
-    (stroke (width 0) (type default))
-  )
   (wire (pts (xy 27.94 160.02) (xy 31.75 160.02))
     (stroke (width 0) (type default))
@@
     (stroke (width 0) (type default))
   )
-  (wire (pts (xy 99.06 181.61) (xy 95.25 181.61))
-    (stroke (width 0) (type default))
-  )
-  (wire (pts (xy 99.06 167.64) (xy 99.06 172.72))
-    (stroke (width 0) (type default))
-  )
   (wire (pts (xy 243.84 29.21) (xy 243.84 33.02))
     (stroke (width 0) (type default))
@@
     (stroke (width 0) (type default))
   )
-  (wire (pts (xy 212.09 111.76) (xy 238.76 111.76))
-    (stroke (width 0) (type default))
-  )
   (wire (pts (xy 252.73 36.83) (xy 252.73 33.02))
     (stroke (width 0) (type default))
@@
     (stroke (width 0) (type default))
   )
-  (wire (pts (xy 86.36 167.64) (xy 99.06 167.64))
-    (stroke (width 0) (type default))
-  )
   (wire (pts (xy 161.29 160.02) (xy 152.4 160.02))
     (stroke (width 0) (type default))
@@
     (stroke (width 0) (type default))
   )
-  (wire (pts (xy 86.36 165.1) (xy 102.87 165.1))
-    (stroke (width 0) (type default))
-  )
-  (wire (pts (xy 215.9 144.78) (xy 212.09 144.78))
-    (stroke (width 0) (type default))
-  )
   (wire (pts (xy 38.1 31.75) (xy 45.72 31.75))
     (stroke (width 0) (type default))
@@
     (stroke (width 0) (type default))
   )
-  (wire (pts (xy 106.68 162.56) (xy 106.68 172.72))
-    (stroke (width 0) (type default))
-  )
   (wire (pts (xy 275.59 41.91) (xy 275.59 48.26))
     (stroke (width 0) (type default))
@@
     (stroke (width 0) (type default))
   )
-  (wire (pts (xy 99.06 167.64) (xy 121.92 167.64))
+  (wire (pts (xy 86.36 167.64) (xy 121.92 167.64))
     (stroke (width 0) (type default))
   )
@@
     (stroke (width 0) (type default))
   )
-  (wire (pts (xy 212.09 134.62) (xy 212.09 111.76))
-    (stroke (width 0) (type default))
-  )
   (wire (pts (xy 161.29 147.32) (xy 152.4 147.32))
     (stroke (width 0) (type default))
@@
     (stroke (width 0) (type default))
   )
-  (wire (pts (xy 102.87 165.1) (xy 102.87 172.72))
-    (stroke (width 0) (type default))
-  )
   (wire (pts (xy 129.54 184.15) (xy 139.7 184.15))
     (stroke (width 0) (type default))
@@
     (stroke (width 0) (type default))
   )
-  (wire (pts (xy 106.68 181.61) (xy 102.87 181.61))
+  (wire (pts (xy 95.25 181.61) (xy 106.68 181.61))
     (stroke (width 0) (type default))
   )
@@
     (stroke (width 0) (type default))
   )
-  (wire (pts (xy 102.87 181.61) (xy 99.06 181.61))
-    (stroke (width 0) (type default))
-  )
-  (wire (pts (xy 212.09 144.78) (xy 212.09 139.7))
-    (stroke (width 0) (type default))
-  )
   (wire (pts (xy 38.1 30.48) (xy 38.1 31.75))
     (stroke (width 0) (type default))
   )
-  (wire (pts (xy 106.68 177.8) (xy 106.68 181.61))
-    (stroke (width 0) (type default))
-  )
-  (wire (pts (xy 86.36 162.56) (xy 106.68 162.56))
+  (wire (pts (xy 86.36 162.56) (xy 121.92 162.56))
     (stroke (width 0) (type default))
   )
@@
   )
   (wire (pts (xy 55.88 49.53) (xy 60.96 49.53))
-    (stroke (width 0) (type default))
-  )
-  (wire (pts (xy 99.06 177.8) (xy 99.06 181.61))
     (stroke (width 0) (type default))
   )
@@
     )
   )
-  (global_label "GIO_5" (shape input) (at 238.76 111.76 0) (fields_autoplaced)
-    (effects (font (size 1.27 1.27)) (justify left))
-    (property "Intersheetrefs" "${INTERSHEET_REFS}" (at 247.1276 111.76 0)
-      (effects (font (size 1.27 1.27)) (justify left) hide)
-    )
-  )
   (global_label "GIO_16" (shape input) (at 238.76 114.3 0) (fields_autoplaced)
     (effects (font (size 1.27 1.27)) (justify left))
@@
     )
   )
-  (symbol (lib_id "Device:R_Small") (at 212.09 137.16 0) (unit 1)
-    (in_bom yes) (on_board yes) (dnp no)
-    (property "Reference" "R?" (at 213.36 134.62 90)
-      (effects (font (size 1.27 1.27)) (justify left))
-    )
-    (property "Value" "10k" (at 210.82 134.62 90)
-      (effects (font (size 1.27 1.27)) (justify left))
-    )
-    (property "Footprint" "Resistor_SMD:R_0603_1608Metric_Pad0.98x0.95mm_HandSolder" (at 212.09 137.16 0)
-      (effects (font (size 1.27 1.27)) hide)
-    )
-    (property "Datasheet" "~" (at 212.09 137.16 0)
-      (effects (font (size 1.27 1.27)) hide)
-    )
-    (pin "1")
-    (pin "2")
-    (instances
-      (project "ESPCARproject"
-        (path "/2f4c7fe4-d81d-42af-a8ed-35cbf01f7760/33af9e60-1f78-4455-a2ff-f16cbea40dbc"
-          (reference "R?") (unit 1)
-        )
-        (path "/2f4c7fe4-d81d-42af-a8ed-35cbf01f7760/ed478ff8-4da3-42ca-8496-863c4885be9c"
-          (reference "R23") (unit 1)
-        )
-      )
-    )
-  )
   (symbol (lib_id "Device:R_Small") (at 36.83 133.35 90) (unit 1)
     (in_bom yes) (on_board yes) (dnp no) (fields_autoplaced)
@@
     )
   )
-  (symbol (lib_id "Device:R_Small") (at 106.68 175.26 0) (unit 1)
-    (in_bom yes) (on_board yes) (dnp no)
-    (property "Reference" "R?" (at 107.95 180.34 90)
-      (effects (font (size 1.27 1.27)) (justify left))
-    )
-    (property "Value" "10k" (at 105.41 180.34 90)
-      (effects (font (size 1.27 1.27)) (justify left))
-    )
-    (property "Footprint" "Resistor_SMD:R_0603_1608Metric_Pad0.98x0.95mm_HandSolder" (at 106.68 175.26 0)
-      (effects (font (size 1.27 1.27)) hide)
-    )
-    (property "Datasheet" "~" (at 106.68 175.26 0)
-      (effects (font (size 1.27 1.27)) hide)
-    )
-    (pin "1")
-    (pin "2")
-    (instances
-      (project "ESPCARproject"
-        (path "/2f4c7fe4-d81d-42af-a8ed-35cbf01f7760/33af9e60-1f78-4455-a2ff-f16cbea40dbc"
-          (reference "R?") (unit 1)
-        )
-        (path "/2f4c7fe4-d81d-42af-a8ed-35cbf01f7760/ed478ff8-4da3-42ca-8496-863c4885be9c"
-          (reference "R19") (unit 1)
-        )
-      )
-    )
-  )
   (symbol (lib_id "power:+3.3V") (at 243.84 22.86 0) (mirror y) (unit 1)
     (in_bom yes) (on_board yes) (dnp no)
@@
         (path "/2f4c7fe4-d81d-42af-a8ed-35cbf01f7760/ed478ff8-4da3-42ca-8496-863c4885be9c"
           (reference "C7") (unit 1)
-        )
-      )
-    )
-  )
-  (symbol (lib_id "Device:R_Small") (at 99.06 175.26 0) (unit 1)
-    (in_bom yes) (on_board yes) (dnp no)
-    (property "Reference" "R?" (at 100.33 180.34 90)
-      (effects (font (size 1.27 1.27)) (justify left))
-    )
-    (property "Value" "10k" (at 97.79 180.34 90)
-      (effects (font (size 1.27 1.27)) (justify left))
-    )
-    (property "Footprint" "Resistor_SMD:R_0603_1608Metric_Pad0.98x0.95mm_HandSolder" (at 99.06 175.26 0)
-      (effects (font (size 1.27 1.27)) hide)
-    )
-    (property "Datasheet" "~" (at 99.06 175.26 0)
-      (effects (font (size 1.27 1.27)) hide)
-    )
-    (pin "1")
-    (pin "2")
-    (instances
-      (project "ESPCARproject"
-        (path "/2f4c7fe4-d81d-42af-a8ed-35cbf01f7760/33af9e60-1f78-4455-a2ff-f16cbea40dbc"
-          (reference "R?") (unit 1)
-        )
-        (path "/2f4c7fe4-d81d-42af-a8ed-35cbf01f7760/ed478ff8-4da3-42ca-8496-863c4885be9c"
-          (reference "R17") (unit 1)
         )
       )
@@
         )
       )
-    )
-  )
-  (symbol (lib_id "Device:R_Small") (at 102.87 175.26 0) (unit 1)
-    (in_bom yes) (on_board yes) (dnp no)
-    (property "Reference" "R?" (at 104.14 172.72 90)
-      (effects (font (size 1.27 1.27)) (justify left))
-    )
-    (property "Value" "10k" (at 101.6 172.72 90)
-      (effects (font (size 1.27 1.27)) (justify left))
-    )
-    (property "Footprint" "Resistor_SMD:R_0603_1608Metric_Pad0.98x0.95mm_HandSolder" (at 102.87 175.26 0)
-      (effects (font (size 1.27 1.27)) hide)
-    )
-    (property "Datasheet" "~" (at 102.87 175.26 0)
-      (effects (font (size 1.27 1.27)) hide)
-    )
-    (pin "1")
-    (pin "2")
-    (instances
-      (project "ESPCARproject"
-        (path "/2f4c7fe4-d81d-42af-a8ed-35cbf01f7760/33af9e60-1f78-4455-a2ff-f16cbea40dbc"
-          (reference "R?") (unit 1)
-        )
-        (path "/2f4c7fe4-d81d-42af-a8ed-35cbf01f7760/ed478ff8-4da3-42ca-8496-863c4885be9c"
-          (reference "R18") (unit 1)
-        )
-      )
